Commit message: removed all the plugins from drone and added zero gravity feauture for drone

File: robots/x3_uav/x3_uav_description/urdf/constants.xacro (robot description, xacro)
@@ -5,7 +5,11 @@
   <xacro:arg name="use_ignition" default="true"/>
   <xacro:arg name="use_plugin" default="true"/>
+  <xacro:arg name="use_plugin_control" default="true"/>
+  <xacro:arg name="zero_gravity" default="true"/>
   <xacro:property name="prefix" value="$(arg prefix)"/>
   <xacro:property name="use_ignition" value="$(arg use_ignition)"/>
   <xacro:property name="use_plugin" value="$(arg use_plugin)"/>
+  <xacro:property name="use_plugin_control" value="$(arg use_plugin_control)"/>
+  <xacro:property name="zero_gravity" value="$(arg zero_gravity)"/>
   <xacro:property name="frame_prefix" value="${prefix + '/' if prefix else ''}"/>
   <xacro:property name="ns_prefix" value="${prefix if prefix else 'x3'}"/>

File: robots/x3_uav/x3_uav_description/urdf/gazebo.xacro (robot description, xacro)
@@ -3,4 +3,5 @@
   <xacro:if value="${use_ignition}">
     <xacro:if value="${use_plugin}">
+    <xacro:if value="${use_plugin_control}">
       <!-- ====================== MOTOR 0 (CCW) ====================== -->
       <gazebo>
@@ -151,4 +152,5 @@
         </plugin>
       </gazebo>
+    </xacro:if>
       <!-- ====================== JOINT STATE PUBLISHER ====================== -->
       <gazebo>
@@ -162,4 +164,31 @@
       </gazebo>
     </xacro:if>
+  <!-- ====================== DISABLE GRAVITY FOR ALL LINKS ====================== -->
+    <xacro:if value="${zero_gravity}">
+      <gazebo reference="${frame_prefix}base_link">
+        <gravity>0</gravity>
+      </gazebo>
+      <gazebo reference="${frame_prefix}rotor_0">
+        <gravity>0</gravity>
+      </gazebo>
+      <gazebo reference="${frame_prefix}rotor_1">
+        <gravity>0</gravity>
+      </gazebo>
+      <gazebo reference="${frame_prefix}rotor_2">
+        <gravity>0</gravity>
+      </gazebo>
+      <gazebo reference="${frame_prefix}rotor_3">
+        <gravity>0</gravity>
+      </gazebo>
+      <gazebo reference="${frame_prefix}imu_link">
+        <gravity>0</gravity>
+      </gazebo>
+      <gazebo reference="${frame_prefix}front_camera_link">
+        <gravity>0</gravity>
+      </gazebo>
+      <gazebo reference="${frame_prefix}bottom_camera_link">
+        <gravity>0</gravity>
+      </gazebo>
+    </xacro:if>
   </xacro:if>
 </robot>

File: robots/x3_uav/x3_uav_description/urdf/sensors.xacro (robot description, xacro)
@@ -5,4 +5,5 @@
 <!-- ============================================ -->
 <xacro:if value="${use_ignition}">
+<xacro:if value="${use_plugin}">
   <!-- ====================== IMU SENSOR ====================== -->
   <!-- <gazebo reference="${frame_prefix}imu_link">
@@ -81,3 +82,4 @@
   </gazebo>
 </xacro:if>
+</xacro:if>
 </robot>
