Commit message: exp rest 5_1 going on along with 103 outside

File: robots/mobile_manipulator/mobile_manipulator_description/urdf/constants.xacro (robot description, xacro)
@@ -11,4 +11,5 @@
   <xacro:arg name="use_hardware" default="false"/>
   <xacro:arg name="use_mock_hardware" default="false"/>
+  <xacro:arg name="plate_colour" default="cyan"/>
   <!-- ============================================ -->
   <!-- PROPERTIES (Converted from arguments) -->
@@ -21,4 +22,5 @@
   <xacro:property name="use_hardware" value="$(arg use_hardware)"/>
   <xacro:property name="use_mock_hardware" value="$(arg use_mock_hardware)"/>
+  <xacro:property name="plate_colour" value="$(arg plate_colour)"/>
   <!-- ============================================ -->
   <!-- NAMESPACE HELPER (for ROS topics and frames) -->

File: robots/mobile_manipulator/mobile_manipulator_description/urdf/joints.xacro (robot description, xacro)
@@ -137,3 +137,9 @@
     <child link="${frame_prefix}caster_wheel"/>
   </joint>
+  <!-- ====================== TOP PLATE FIXED JOINT ====================== -->
+  <joint name="${frame_prefix}top_plate_joint" type="fixed">
+    <parent link="${frame_prefix}base_link"/>
+    <child  link="${frame_prefix}top_plate_link"/>
+    <origin xyz="0 0 0.125" rpy="0 0 0"/>
+  </joint>
 </robot>

File: robots/mobile_manipulator/mobile_manipulator_description/urdf/links.xacro (robot description, xacro)
@@ -503,3 +503,29 @@
     </collision>
   </link>
+  <link name="${frame_prefix}top_plate_link">
+    <!-- Visual -->
+    <visual>
+      <origin xyz="0 0 0" rpy="0 0 0"/>
+      <geometry>
+        <box size="0.35 0.35 0.01"/>  <!-- 22cm × 22cm × 1cm -->
+      </geometry>
+       <material name="cyan"/>
+    </visual>
+    <!-- Collision -->
+    <collision>
+      <origin xyz="0 0 0" rpy="0 0 0"/>
+      <geometry>
+        <box size="0.35 0.35 0.01"/>
+      </geometry>
+    </collision>
+    <!-- Inertial -->
+    <inertial>
+      <origin xyz="0 0 0" rpy="0 0 0"/>
+      <mass value="0.3"/>  <!-- 300 grams -->
+      <inertia
+        ixx="0.0005" ixy="0" ixz="0"
+        iyy="0.0005" iyz="0"
+        izz="0.0004"/>
+    </inertial>
+  </link>
 </robot>

File: robots/x3_uav/x3_uav_description/urdf/sensors.xacro (robot description, xacro)
@@ -52,5 +52,5 @@
     <sensor name="${frame_prefix}bottom_rgbd_camera" type="rgbd_camera">
       <always_on>true</always_on>
-    <update_rate>5</update_rate>
+    <update_rate>10</update_rate>
     <visualize>false</visualize>
       <topic>/${frame_prefix}bottom_camera</topic>
