Commit message: team goal status fixed, yahboom vy fixed

File: robots/yahboom/yahboom_rosmaster_description/urdf/control/velocity_control_plugin.urdf.xacro (robot description, xacro)
@@ -8,10 +8,27 @@
                 filename="ignition-gazebo-velocity-control-system"
                 name="ignition::gazebo::systems::VelocityControl">
-                <!-- <topic>/${frame_prefix}cmd_vel</topic> -->
                 <namespace>${frame_prefix}</namespace>
+                <!-- <link_name>${frame_prefix}base_footprint</link_name> -->
                 <topic>${frame_prefix}cmd_vel</topic>
                 <initial_linear>0 0 0</initial_linear>
                 <initial_angular>0 0 0</initial_angular>
             </plugin>
+            <!-- <plugin
+                filename="libignition-gazebo-mecanum-drive-system.so"
+                name="ignition::gazebo::systems::MecanumDrive">
+                <front_left_joint>${frame_prefix}front_left_wheel_joint</front_left_joint>
+                <front_right_joint>${frame_prefix}front_right_wheel_joint</front_right_joint>
+                <back_left_joint>${frame_prefix}back_left_wheel_joint</back_left_joint>
+                <back_right_joint>${frame_prefix}back_right_wheel_joint</back_right_joint>
+                <wheel_separation>0.169</wheel_separation>
+                <wheelbase>0.16</wheelbase>
+                <wheel_radius>0.0325</wheel_radius>
+                <topic>${frame_prefix}cmd_vel</topic> -->
+                <!-- <odom_topic>${frame_prefix}odom</odom_topic> -->
+                <!-- <tf_topic>/tf</tf_topic> -->
+                <!-- <frame_id>${frame_prefix}odom</frame_id> -->
+                <!-- <child_frame_id>${frame_prefix}base_footprint</child_frame_id> -->
+                <!-- <odom_publish_frequency>50</odom_publish_frequency> -->
+            <!-- </plugin> -->
             <!-- Fortress odom publisher -->
             <plugin

File: robots/yahboom/yahboom_rosmaster_description/urdf/mech/mecanum_wheel.urdf.xacro (robot description, xacro)
@@ -4,5 +4,5 @@
   <xacro:property name="wheel_separation" value="0.169" />
   <xacro:property name="wheel_width" value="0.03040" />
-  <xacro:property name="wheel_mass" value="9.1" />
+  <xacro:property name="wheel_mass" value="0.15" />
   <xacro:property name="wheel_xoff" value="0.08" />
   <xacro:property name="wheel_yoff" value="-0.01" />
@@ -39,22 +39,27 @@
       <origin xyz="${x_reflect*wheel_xoff} ${y_reflect*(wheel_separation/2+wheel_yoff)} ${-wheel_radius}" rpy="0 0 0"/>
     </joint>
-    <gazebo reference="${frame_prefix}${side}_wheel_link">
-      <surface>
-        <friction>
-          <ode>
-              <mu>1.0</mu>
-              <mu2>0.0</mu2>
-          </ode>
-        </friction>
-      </surface>
-      <visual>
-          <material>
-              <ambient>0.2 0.2 0.2 1.0</ambient>
-              <diffuse>0.2 0.2 0.2 1.0</diffuse>
-              <specular>0.2 0.2 0.2 1.0</specular>
-              <emissive>0.0 0.0 0.0 0.0</emissive>
-          </material>
-      </visual>
-  </gazebo>
+<gazebo reference="${frame_prefix}${side}_wheel_link">
+    <mu1>0.0</mu1>
+    <mu2>0.0</mu2>
+    <kp>0</kp>
+    <kd>0</kd>
+    <collide_without_contact>false</collide_without_contact>
+    <collision>
+        <surface>
+            <friction>
+                <ode>
+                    <mu>0.0</mu>
+                    <mu2>0.0</mu2>
+                </ode>
+            </friction>
+            <contact>
+                <ode>
+                    <kp>0</kp>
+                    <kd>0</kd>
+                </ode>
+            </contact>
+        </surface>
+    </collision>
+</gazebo>
   </xacro:macro>
 </robot>
